Commit message: att sensores

File: src/ugv_simulation/robots_description/sensors/imu_sensor.urdf.xacro (robot description, xacro)
@@ -1,18 +1,18 @@
 <robot xmlns:xacro="http://ros.org/wiki/xacro">
     <xacro:macro name="imu_sensor">
-        <link name="imu"/>
+        <link name="imu_link"/>
         <joint name="imu_to_body" type="fixed">
-        <parent link="body"/>
-        <child link="imu"/>
-        <origin xyz="0 0 0" rpy="0 0 0"/>
+            <parent link="body"/>
+            <child link="imu_link"/>
+            <origin xyz="0 0 0" rpy="0 0 0"/>
         </joint>
-        <gazebo reference="imu">
-            <gravity>true</gravity>
+       <gazebo reference="imu_link">
+        <gravity>true</gravity>
             <sensor name="imu_sensor" type="imu">
                 <always_on>true</always_on>
                 <update_rate>20</update_rate>
-                <visualize>true</visualize>
+                <visualize>false</visualize>
                 <topic>__default_topic__</topic>
-                <plugin name="imu_plugin" filename="libgazebo_ros_imu_sensor.so">
+                <plugin filename="libgazebo_ros_imu_sensor.so" name="imu_plugin">
                     <ros>
                         <remapping>~/out:=imu/data</remapping>
@@ -24,6 +24,4 @@
                     <xyzOffset>0 0 0</xyzOffset>
                     <rpyOffset>0 0 0</rpyOffset>
-                    <frameName>imu</frameName>
-                    <initialOrientationAsReference>false</initialOrientationAsReference>
                 </plugin>
                 <pose>0 0 0 0 0 0</pose>

File: src/ugv_simulation/robots_description/sensors/laser_sensor.urdf.xacro (robot description, xacro)
@@ -3,37 +3,27 @@
     <xacro:macro name="laser_sensor" params="update_rate ray_count min_angle max_angle min_range max_range frame_id topic_name">
         <link name="${frame_id}">
-        <visual>
-            <origin xyz="0 0 -0.025" rpy="0 0 ${M_PI/2}"/>
-            <geometry>
-                <mesh filename="file:///$(find ugv_simulation)/robots_description/meshes/rplidar.dae"/>
-            </geometry>
-            <material name="green">
-                <color rgba="0.003 0.639 0.223 1.0"/>
-            </material>
-        </visual>
-        <collision>
-            <origin xyz="0.003 -0.003 -0.027" rpy="0 0 ${M_PI/2}"/>
-            <geometry>
-                <cylinder radius="0.0375" length="0.05"/>
-            </geometry>
-        </collision>
-        <inertial>
-            <origin xyz="0 0 0" rpy="0 0 0"/>
-            <mass value="0.1"/>
-            <inertia ixx="${(2/5) * 0.1 * (0.0375 * 0.0375)}" ixy="0" ixz="0"
-                    iyy="${(2/5) * 0.1 * (0.0375 * 0.0375)}" iyz="0"
-                    izz="${(2/5) * 0.1 * (0.0375 * 0.0375)}" />
+            <visual>
+                <origin xyz="0 0 -0.025" rpy="0 0 ${M_PI/2}"/>
+                <geometry>
+                    <mesh filename="file:///$(find oni_claw_gazebo)/robot_description/meshes/rplidar.dae"/>
+                </geometry>
+                <material name="white">
+                    <color rgba="1 1 1 1"/>
+                </material>
+            </visual>
+            <collision>
+                <origin xyz="0.003 -0.003 -0.027" rpy="0 0 ${M_PI/2}"/>
+                <geometry>
+                    <cylinder radius="0.0375" length="0.04"/>
+                </geometry>
+            </collision>
+            <inertial>
+                <origin xyz="0 0 0" rpy="0 0 0"/>
+                <mass value="0.1"/>
+                <inertia ixx="${(2/5) * 0.1 * (0.0375 * 0.0375)}" ixy="0" ixz="0"
+                        iyy="${(2/5) * 0.1 * (0.0375 * 0.0375)}" iyz="0"
+                        izz="${(2/5) * 0.1 * (0.0375 * 0.0375)}" />
             </inertial>
         </link>
-        <gazebo reference="${frame_id}">
-        <visual>
-            <material>
-            <ambient>0.003 0.639 0.223 1.0</ambient>
-            <diffuse>0.003 0.639 0.223 1.0</diffuse>
-            <specular>0.003 0.639 0.223 1.0</specular>
-            <emissive>0.0 0.0 0.0 0.0</emissive>
-            </material>
-        </visual>
-        </gazebo>
         <joint name="${frame_id}_to_body" type="fixed">
             <parent link="body"/>
@@ -42,36 +32,48 @@
         </joint>
         <gazebo reference="${frame_id}">
-        <sensor type="ray" name="${frame_id}_head_hokuyo_sensor">
-            <always_on>true</always_on>
-            <update_rate>${update_rate}</update_rate>
-            <pose>0 0 0 0 0 0</pose>
-            <visualize>false</visualize>
-            <ray>
-            <scan>
-                <horizontal>
-                <samples>${ray_count}</samples>
-                <resolution>1</resolution>
-                <min_angle>${min_angle}</min_angle>
-                <max_angle>${max_angle}</max_angle>
-                </horizontal>
-            </scan>
-            <range>
-                <min>${min_range}</min>
-                <max>${max_range}</max>
-                <resolution>0.01</resolution>
-            </range>
-            </ray>
-            <plugin name="${frame_id}_gazebo_ros_head_hokuyo_controller" filename="libgazebo_ros_ray_sensor.so">
-            <ros>
-                <remapping>~/out:=${topic_name}</remapping>
-            </ros>
-            <output_type>sensor_msgs/LaserScan</output_type>
-            <alwaysOn>true</alwaysOn>
-            <updateRate>${update_rate}</updateRate>
-            <topicName>${topic_name}</topicName>
-            <frame_name>${frame_id}</frame_name>
-            <output_type>sensor_msgs/LaserScan</output_type>
-            </plugin>
-        </sensor>
+            <visual>
+                <material>
+                    <ambient>0.003 0.639 0.223 1.0</ambient>
+                    <diffuse>0.003 0.639 0.223 1.0</diffuse>
+                    <specular>0.003 0.639 0.223 1.0</specular>
+                    <emissive>0.0 0.0 0.0 0.0</emissive>
+                </material>
+            </visual>
+        </gazebo>
+        <gazebo reference="${frame_id}">
+            <sensor type="ray" name="${frame_id}_head_hokuyo_sensor">
+                <always_on>true</always_on>
+                <update_rate>${update_rate}</update_rate>
+                <pose>0 0 0 0 0 0</pose>
+                <visualize>false</visualize>
+                <ray>
+                    <scan>
+                        <horizontal>
+                        <samples>${ray_count}</samples>
+                        <resolution>1</resolution>
+                        <min_angle>${min_angle}</min_angle>
+                        <max_angle>${max_angle}</max_angle>
+                        </horizontal>
+                    </scan>
+                    <range>
+                        <min>${min_range}</min>
+                        <max>${max_range}</max>
+                        <resolution>0.01</resolution>
+                    </range>
+                    <noise>
+                        <type>gaussian</type>
+                        <mean>0.0</mean>
+                        <stddev>0.01</stddev>
+                    </noise>
+                </ray>
+                <plugin name="${frame_id}_gazebo_ros_head_hokuyo_controller" filename="libgazebo_ros_ray_sensor.so">
+                    <ros>
+                        <remapping>~/out:=${topic_name}</remapping>
+                    </ros>
+                    <output_type>sensor_msgs/LaserScan</output_type>
+                    <topicName>${topic_name}</topicName>
+                    <frame_name>${frame_id}</frame_name>
+                </plugin>
+            </sensor>
         </gazebo>
   </xacro:macro>
