Commit message: reorganização dos pacotes e config do sistema

File: src/ugv_robots_descriptions/robots_description/controller/omni_drive.urdf.xacro (robot description, xacro)
@@ -3,9 +3,12 @@
         <gazebo>
             <plugin name="omni_drive_controller" filename="libgazebo_ros_planar_move.so">
+                <ros>
+                    <argument>odom:=odom/unfiltered</argument>
+                </ros>
                 <command_topic>cmd_vel</command_topic>
-                <odometry_topic>odom/unfiltered</odometry_topic>
+                <odometry_topic>odom/unfiltered/</odometry_topic>
                 <odometry_frame>odom</odometry_frame>
                 <odometry_rate>20.0</odometry_rate>
-                <robot_base_frame>base_footprint</robot_base_frame>
+                <robot_base_frame>base_link</robot_base_frame>
                 <publish_odom>true</publish_odom>
                 <publish_odom_tf>false</publish_odom_tf>

File: src/ugv_robots_descriptions/robots_description/sensors/laser_sensor.urdf.xacro (robot description, xacro)
@@ -6,5 +6,5 @@
                 <origin xyz="0 0 -0.025" rpy="0 0 ${M_PI/2}"/>
                 <geometry>
-                    <mesh filename="file:///$(find oni_claw_gazebo)/robot_description/meshes/rplidar.dae"/>
+                    <mesh filename="file:///$(find ugv_robots_description)/robot_description/meshes/rplidar.dae"/>
                 </geometry>
                 <material name="white">
@@ -26,6 +26,6 @@
             </inertial>
         </link>
-        <joint name="${frame_id}_to_body" type="fixed">
-            <parent link="body"/>
+        <joint name="${frame_id}_to_base_link" type="fixed">
+            <parent link="base_link"/>
             <child link="${frame_id}"/>
             <origin xyz="-0.0475 0 0.075" rpy="0 0 0"/>
@@ -74,4 +74,5 @@
                     <topicName>${topic_name}</topicName>
                     <frame_name>${frame_id}</frame_name>
+                    <output_type>sensor_msgs/LaserScan</output_type>
                 </plugin>
             </sensor>
