Commit message: Adicionando o launchers e alguns arquivos do l1br

File: src/ugv_robots_descriptions/robots_description/oni.urdf.xacro (robot description, xacro)
@@ -53,5 +53,5 @@
             <origin xyz="0 0 0" rpy="0 0 -${pi/2}"/>
             <geometry>
-                <mesh filename="file:///$(find ugv_robots_description)/robot_description/meshes/oni_meshes/body_OC.dae"/>
+                <mesh filename="file:///$(find ugv_robots_description)/robot_description/meshes/oni_meshes/chassis.dae"/>
             </geometry>
         </visual>
@@ -59,5 +59,5 @@
             <origin xyz="0 0 0" rpy="0 0 -${pi/2}"/>
             <geometry>
-                <mesh filename="file:///$(find ugv_robots_description)/robot_description/meshes/oni_meshes/body_OC.dae"/>
+                <mesh filename="file:///$(find ugv_robots_description)/robot_description/meshes/oni_meshes/chassis.dae"/>
             </geometry>
         </collision>
@@ -104,6 +104,7 @@
         min_range="0.12"
         max_range="8.0"
-        frame_id="lidar_link"
-        topic_name="scan"
+        pos_x="-0.0475"
+        pos_y="0"
+        pos_z="0.075"
     />
     <xacro:omni_drive_controller/>

File: src/ugv_robots_descriptions/robots_description/sensors/laser_sensor.urdf.xacro (robot description, xacro)
@@ -1,6 +1,6 @@
 <robot xmlns:xacro="http://ros.org/wiki/xacro">
     <xacro:property name="M_PI" value="3.1415926535897931" />
-    <xacro:macro name="laser_sensor" params="update_rate ray_count min_angle max_angle min_range max_range frame_id topic_name">
-        <link name="${frame_id}">
+    <xacro:macro name="laser_sensor" params="update_rate ray_count min_angle max_angle min_range max_range pos_x pos_y pos_z">
+        <link name="base_link">
             <visual>
                 <origin xyz="0 0 -0.025" rpy="0 0 ${M_PI/2}"/>
@@ -26,10 +26,10 @@
             </inertial>
         </link>
-        <joint name="${frame_id}_to_base_link" type="fixed">
+        <joint name="base_link_to_base_link" type="fixed">
             <parent link="base_link"/>
-            <child link="${frame_id}"/>
+            <child link="base_link"/>
             <origin xyz="-0.0475 0 0.075" rpy="0 0 0"/>
         </joint>
-        <gazebo reference="${frame_id}">
+        <gazebo reference="base_link">
             <visual>
                 <material>
@@ -41,6 +41,6 @@
             </visual>
         </gazebo>
-        <gazebo reference="${frame_id}">
-            <sensor type="ray" name="${frame_id}_head_hokuyo_sensor">
+        <gazebo reference="base_link">
+            <sensor type="ray" name="base_link_head_hokuyo_sensor">
                 <always_on>true</always_on>
                 <update_rate>${update_rate}</update_rate>
@@ -67,11 +67,11 @@
                     </noise>
                 </ray>
-                <plugin name="${frame_id}_gazebo_ros_head_hokuyo_controller" filename="libgazebo_ros_ray_sensor.so">
+                <plugin name="base_link_gazebo_ros_head_hokuyo_controller" filename="libgazebo_ros_ray_sensor.so">
                     <ros>
-                        <remapping>~/out:=${topic_name}</remapping>
+                        <remapping>~/out:=scan</remapping>
                     </ros>
                     <output_type>sensor_msgs/LaserScan</output_type>
-                    <topicName>${topic_name}</topicName>
-                    <frame_name>${frame_id}</frame_name>
+                    <topicName>scan</topicName>
+                    <frame_name>base_link</frame_name>
                     <output_type>sensor_msgs/LaserScan</output_type>
                 </plugin>

Commit message: Systema pronto para os primeiros testes

File: src/ugv_robots_descriptions/robots_description/oni.urdf.xacro (robot description, xacro)
@@ -4,4 +4,5 @@
     <xacro:include filename="sensors/laser_sensor.urdf.xacro"/>
     <xacro:include filename="controller/omni_drive.urdf.xacro"/>
+    <xacro:property name="chassis" value="file:///$(find ugv_robots_description)/robot_description/meshes/oni_meshes/chassis.dae">
     <xacro:property name="wheel_radius" value="0.033"/>
     <xacro:property name="wheel_width" value="0.026"/>
@@ -10,5 +11,38 @@
     <xacro:property name="wheel_zoff" value="-0.014"/>
     <xacro:property name="wheel_mass" value="0.3"/>
-    <xacro:macro name="mecanum_wheel" params="side x_reflect y_reflect orientation_z mesh">
+    <xacro:macro name="base_link">
+        <link name="base_link">
+            <visual>
+                <origin xyz="0 0 0" rpy="0 0 -${pi/2}"/>
+                <geometry>
+                    <mesh filename="${chassis}"/>
+                </geometry>
+            </visual>
+            <collision>
+                <origin xyz="0 0 0" rpy="0 0 -${pi/2}"/>
+                <geometry>
+                    <mesh filename="${chassis}"/>
+                </geometry>
+            </collision>
+            <inertial>
+                <mass value="0.8"/>
+                <origin xyz="0 0 0" rpy="0 0 0" />
+                <inertia ixx="0.0029" ixy="0.0" ixz="0.0" iyy="0.0029" iyz="0.0" izz="0.00533"/>
+            </inertial>
+        </link>
+        <gazebo reference="base_link">
+            <mu1>0.3<mu1/>
+            <mu2>0.3<mu2/>
+            <kp>1000000.0<kp/>
+            <kd>100<kd/>
+        </gazebo>
+        <link name="base_footprint"/>
+        <joint name="base_footprint_to_base_link" type="fixed">
+            <parent link="base_link"/>
+            <child link="base_footprint"/>
+            <origin xyz="0.0 0.0 ${-wheel_radius - wheel_zoff}" rpy="0 0 0"/>
+        </joint>
+    </xacro:macro>
+    <xacro:macro name="mecanum_wheel_link" params="side x_reflect y_reflect orientation_z mesh">
         <link name="${side}_wheel_link">
         <visual>
@@ -35,4 +69,6 @@
             <mu1>0.01</mu1>
             <mu2>0.01</mu2>
+            <kp>1000000.0</kp>
+            <kd>100.0</kd>
         </gazebo>
         <joint name="${side}_wheel_to_base_link" type="continuous">
@@ -43,30 +79,6 @@
         </joint>
     </xacro:macro>
-    <link name="base_footprint"/>
-    <joint name="base_footprint_to_base_link" type="fixed">
-        <parent link="base_link"/>
-        <child link="base_footprint"/>
-        <origin xyz="0.0 0.0 ${-wheel_radius - wheel_zoff}" rpy="0 0 0"/>
-    </joint>
-    <link name="base_link">
-        <visual>
-            <origin xyz="0 0 0" rpy="0 0 -${pi/2}"/>
-            <geometry>
-                <mesh filename="file:///$(find ugv_robots_description)/robot_description/meshes/oni_meshes/chassis.dae"/>
-            </geometry>
-        </visual>
-        <collision>
-            <origin xyz="0 0 0" rpy="0 0 -${pi/2}"/>
-            <geometry>
-                <mesh filename="file:///$(find ugv_robots_description)/robot_description/meshes/oni_meshes/chassis.dae"/>
-            </geometry>
-        </collision>
-        <inertial>
-            <mass value="0.8"/>
-            <origin xyz="0 0 0" rpy="0 0 0" />
-            <inertia ixx="0.0029" ixy="0.0" ixz="0.0" iyy="0.0029" iyz="0.0" izz="0.00533"/>
-        </inertial>
-    </link>
-    <xacro:mecanum_wheel
+    <xacro:base_link>
+    <xacro:mecanum_wheel_link
         side="front_right"
         x_reflect="1"
@@ -75,5 +87,5 @@
         mesh="file:///$(find ugv_robots_description)/robot_description/meshes/oni_meshes/fr_wheel.dae"
     />
-    <xacro:mecanum_wheel
+    <xacro:mecanum_wheel_link
         side="front_left"
         x_reflect="1"
@@ -82,5 +94,5 @@
         mesh="file:///$(find ugv_robots_description)/robot_description/meshes/oni_meshes/fl_wheel.dae"
     />
-    <xacro:mecanum_wheel
+    <xacro:mecanum_wheel_link
         side="back_right"
         x_reflect="-1"
@@ -89,5 +101,5 @@
         mesh="file:///$(find ugv_robots_description)/robot_description/meshes/oni_meshes/fr_wheel.dae"
     />
-    <xacro:mecanum_wheel
+    <xacro:mecanum_wheel_link
         side="back_left"
         x_reflect="-1"
