Commit message: Consertado posicionamento do lidar nos robôs

File: install/ugv_robots_descriptions/share/ugv_robots_descriptions/robots_description/sensors/laser_sensor.urdf.xacro (robot description, xacro)
@@ -29,7 +29,7 @@
             <parent link="base_link"/>
             <child link="laser_link"/>
-            <origin xyz="-0.0475 0 0.075" rpy="0 0 0"/>
+            <origin xyz="${pos_x} ${pos_y} ${pos_z}" rpy="0 0 0"/>
         </joint>
-        <gazebo reference="base_link">
+        <gazebo reference="laser_link">
             <visual>
                 <material>
@@ -41,5 +41,5 @@
             </visual>
         </gazebo>
-        <gazebo reference="base_link">
+        <gazebo reference="laser_link">
             <sensor type="ray" name="base_link_head_hokuyo_sensor">
                 <always_on>true</always_on>
@@ -73,5 +73,5 @@
                     <output_type>sensor_msgs/LaserScan</output_type>
                     <topicName>scan</topicName>
-                    <frame_name>lidar_link</frame_name>
+                    <frame_name>laser_link</frame_name>
                     <output_type>sensor_msgs/LaserScan</output_type>
                 </plugin>
