Commit message: Refatorado launcher do mapa, consertado fisica das rodas do omnidirecional, consertado sh para instalação de ferramentas necessárias

File: ugv_robots_descriptions/robots_description/oni.urdf.xacro (robot description, xacro)
@@ -67,11 +67,12 @@
         </link>
         <gazebo reference="${side}_wheel_link">
-            <mu1>1.0</mu1>
-            <mu2>1.0</mu2>
+            <selfCollide>false</selfCollide>
+            <mu1>0.03</mu1>
+            <mu2>0.03</mu2>
             <kp>1000000.0</kp>
             <kd>100.0</kd>
         </gazebo>
         <joint name="${side}_wheel_to_base_link" type="continuous">
-            <axis xyz="1 0 0" />
+            <axis xyz="0 1 0" />
             <parent link="base_link"/>
             <child link="${side}_wheel_link"/>
