Commit message: Att modelo dos robôs

File: ugv_robots_descriptions/robots_description/l1br.urdf.xacro (robot description, xacro)
@@ -7,23 +7,33 @@
     <xacro:property name="base_length" value="0.77"/>
     <xacro:property name="base_height" value="0.13"/>
+    <xacro:property name="base_mass" value="2.4"/>
     <xacro:property name="wheel_radius" value="0.0675"/>
     <xacro:property name="wheel_width" value="0.04"/>
+    <xacro:property name="wheel_mass" value="1"/>
     <xacro:property name="caster_wheel_radius" value="0.01"/>
+    <xacro:property name="caster_wheel_radius_visual" value="0.001"/>
+    <xacro:property name="caster_wheel_mass" value="0.005"/>
     <xacro:property name="tray_radius" value="0.2"/>
-    <xacro:property name="tray_width" value="0.041"/>
+    <xacro:property name="tray_width" value="0.03"/>
+    <xacro:property name="piston_cylinder_width" value="0.15"/>
+    <xacro:property name="piston_cylinder_radius" value="0.015"/>
+    <xacro:property name="piston_cylinder_mass" value="0.2"/>
+    <xacro:property name="piston_base_width" value="0.01"/>
+    <xacro:property name="piston_base_radius" value="0.08"/>
+    <xacro:property name="piston_base_mass" value="0.2"/>
     <xacro:macro name="base_link">
         <link name="base_footprint">
         </link>
         <gazebo reference="base_link">
-            <mu1 value="0.3" />
-            <mu2 value="0.3" />
-            <kp value="1000000.0" />
-            <kd value="100" />
-            <fdir1 value="0 0 0" />
+        <mu1 value="0.3" />
+        <mu2 value="0.3" />
+        <kp value="1000000.0" />
+        <kd value="100" />
+        <fdir1 value="0 0 0" />
         </gazebo>
         <joint name="base_joint" type="fixed">
-            <parent link="base_link"/>
-            <child link="base_footprint" />
-            <origin xyz="0.0 0.0 -0.0793" rpy="0 0 3.14"/>
+        <parent link="base_link"/>
+        <child link="base_footprint" />
+        <origin xyz="0.0 0.0 -0.0793" rpy="0 0 3.14"/>
         </joint>
         <link name="base_link">
@@ -31,5 +41,5 @@
             <origin xyz="0  0  0" rpy="0 0 0"/>
             <geometry>
-            <mesh filename="file:///$(find ugv_robots_descriptions)/robots_description/meshes/l1br_meshes/chassis.dae" />
+            <mesh filename="file:///$(find ugv_robots_description)/meshes/l1br_meshes/chassis.dae" />
             </geometry>
         </visual>
@@ -42,5 +52,5 @@
         <inertial>
             <origin xyz="0  0  0.0" rpy="0 0 1.57"/>
-            <mass value="2.4"/>
+            <mass value="${base_mass}"/>
             <inertia ixx="0.12196" ixy="0.0" ixz="0.0"
                     iyy="0.04756" iyz="0.0"
@@ -58,6 +68,6 @@
         <gazebo reference="${prefix}">
             <selfCollide>false</selfCollide>
-            <mu1>1.0</mu1>
-            <mu2>1.0</mu2>
+            <mu1>1.5</mu1>
+            <mu2>1.5</mu2>
             <kp>1000000.0</kp>
             <kd>100.0</kd>
@@ -65,9 +75,9 @@
         <link name="${prefix}">
             <inertial>
-                <mass value="1" />
+                <mass value="${wheel_mass}" />
                 <origin rpy="0 1.57 0" xyz="0 0 0" />
-                <inertia ixx="${(2/5) * 1 * (wheel_radius * wheel_radius)}" ixy="0" ixz="0"
-                         iyy="${(2/5) * 1 * (wheel_radius * wheel_radius)}" iyz="0"
-                         izz="${(2/5) * 1 * (wheel_radius * wheel_radius)}" />
+                <inertia ixx="${(2/5) * wheel_mass * (wheel_radius * wheel_radius)}" ixy="0" ixz="0"
+                         iyy="${(2/5) * wheel_mass * (wheel_radius * wheel_radius)}" iyz="0"
+                         izz="${(2/5) * wheel_mass * (wheel_radius * wheel_radius)}" />
             </inertial>
             <collision name="${prefix}_collision">
@@ -80,5 +90,5 @@
                 <origin rpy="0 0 0" xyz="0 0 0" />
                 <geometry>
-                    <mesh filename="file:///$(find ugv_robots_descriptions)/robots_description/meshes/l1br_meshes/wheel.dae" scale="1 1 1" />
+                    <mesh filename="file:///$(find ugv_robots_description)/meshes/wheel.dae" scale="1 1 1" />
                 </geometry>
             </visual>
@@ -94,6 +104,6 @@
         <gazebo reference="${prefix}">
             <selfCollide>false</selfCollide>
-            <mu1>0.09</mu1>
-            <mu2>0.09</mu2>
+            <mu1>0.2</mu1>
+            <mu2>0.2</mu2>
             <kp>10000000.0</kp>
             <kd>10000.0</kd>
@@ -101,9 +111,9 @@
         <link name="${prefix}">
             <inertial>
-                <mass value="0.005" />
-                <origin rpy="0 0 0" xyz="0 0 0" />
-                <inertia ixx="${(2/5) * 0.005 * (caster_wheel_radius * caster_wheel_radius)}" ixy="0" ixz="0"
-                         iyy="${(2/5) * 0.005 * (caster_wheel_radius * caster_wheel_radius)}" iyz="0"
-                         izz="${(2/5) * 0.005 * (caster_wheel_radius * caster_wheel_radius)}" />
+                <mass value="${caster_wheel_mass}" />
+                <origin rpy="0 0 0" xyz="0 0 0" />
+                <inertia ixx="${(2/5) * caster_wheel_mass * (caster_wheel_radius * caster_wheel_radius)}" ixy="0" ixz="0"
+                         iyy="${(2/5) * caster_wheel_mass * (caster_wheel_radius * caster_wheel_radius)}" iyz="0"
+                         izz="${(2/5) * caster_wheel_mass * (caster_wheel_radius * caster_wheel_radius)}" />
             </inertial>
             <collision name="${prefix}_collision">
@@ -116,5 +126,5 @@
                 <origin rpy="0 0 0" xyz="0 0 0" />
                 <geometry>
-                    <sphere radius="${caster_wheel_radius}"/>
+                    <sphere radius="${caster_wheel_radius_visual}"/>
                 </geometry>
             </visual>
@@ -126,9 +136,9 @@
             <origin xyz="0 0 0.0118" rpy="0 0 0"/>
             <geometry>
-                <mesh filename="file:///$(find ugv_robots_descriptions)/robots_description/meshes/l1br_meshes/tray.dae" scale="1 1 1"/>
+                <mesh filename="file:///$(find l1br)/meshes/ELV_conjuntocompleto.dae" scale="1 1 1"/>
             </geometry>
         </visual>
         <collision name="tray_collision">
-            <origin xyz="0 -0.015047 0.1" rpy="0 0 0"/>
+            <origin xyz="0 0 0.105" rpy="0 0 0"/>
             <geometry>
             <cylinder length="${tray_width}" radius="${tray_radius}"/>
@@ -138,13 +148,105 @@
             <mass value="0.5" />
             <origin rpy="0 0 0" xyz="0 0 0" />
-            <inertia ixx="0.0" ixy="0.0" ixz="0.0"
-                    iyy="0.0" iyz="0.0"
-                    izz="0.0" />
+            <inertia ixx="${(2/5) * 0.5 * (tray_radius * tray_radius)}" ixy="0.0" ixz="0.0"
+                    iyy="${(2/5) * 0.5 * (tray_radius * tray_radius)}" iyz="0.0"
+                    izz="${(2/5) * 0.5 * (tray_radius * tray_radius)}" />
         </inertial>
         </link>
-        <joint name="joint_tray" type="fixed">
+        <gazebo reference="tray_link">
+            <selfCollide>true</selfCollide>
+            <mu1 value="1.5" />
+            <mu2 value="1.5" />
+            <kp value="10000000.0" />
+            <kd value="10000" />
+            <fdir1 value="0 0 0" />
+        </gazebo>
+        <!-- <joint name="joint_prismatic_tray" type="prismatic"> -->
+                <!-- <parent link="base_link" /> -->
+                <!-- <child link="tray_link" /> -->
+                <!-- <origin rpy="0 0 0" xyz="0 0.015047 0" /> -->
+                <!-- <axis xyz="0 0 1"/> -->
+                <!-- <limit effort="1000.0" lower="0" upper="0.3" velocity="0.5"/> -->
+        <!-- </joint> -->
+        <joint name="joint_tray" type="continuous">
+                <parent link="piston_base" />
+                <child link="tray_link" />
+                <origin rpy="0 0 0" xyz="0 0 -0.08" />
+                <axis xyz="0 0 1"/>
+        </joint>
+    </xacro:macro>
+    <xacro:macro name="piston_link">
+        <gazebo reference="piston_cylinder">
+            <selfCollide>false</selfCollide>
+            <mu1>0.1</mu1>
+            <mu2>0.1</mu2>
+            <kp>10000000.0</kp>
+            <kd>10000.0</kd>
+        </gazebo>
+        <link name="piston_cylinder">
+            <visual name="piston_cylinder_visual">
+                <origin xyz="0 0 0" rpy="0 0 0"/>
+                <geometry>
+                    <cylinder length="${piston_cylinder_width}" radius="${piston_cylinder_radius}"/>
+                </geometry>
+                <material name="grey">
+                    <color rgba="0.2 0.2 0.2 1.0"/>
+                </material>
+            </visual>
+            <!-- <collision name="piston_cylinder_collision"> -->
+                <!-- <origin xyz="0 0 0" rpy="0 0 0"/> -->
+                <!-- <geometry> -->
+                    <!-- <cylinder length="${piston_cylinder_width}" radius="${piston_cylinder_radius}"/> -->
+                <!-- </geometry> -->
+            <!-- </collision> -->
+            <inertial>
+                <mass value="${piston_cylinder_mass}" />
+                <origin rpy="0 0 0" xyz="0 0 0" />
+                <inertia ixx="${(2/5) * piston_cylinder_mass * (piston_cylinder_radius * piston_cylinder_radius)}" ixy="0.0" ixz="0.0"
+                        iyy="${(2/5) * piston_cylinder_mass * (piston_cylinder_radius * piston_cylinder_radius)}" iyz="0.0"
+                        izz="${(2/5) * piston_cylinder_mass * (piston_cylinder_radius * piston_cylinder_radius)}" />
+            </inertial>
+        </link>
+        <joint name="joint_piston_cylinder" type="prismatic">
                 <parent link="base_link" />
-                <child link="tray_link" />
-                <origin rpy="0 0 0" xyz="0 0.015047 0" />
+                <child link="piston_cylinder" />
+                <origin rpy="0 0 0" xyz="0 0 0.02" />
+                <axis xyz="0 0 1"/>
+                <limit effort="1000.0" lower="0" upper="0.12" velocity="0.3"/>
+        </joint>
+        <gazebo reference="piston_base">
+            <selfCollide>false</selfCollide>
+            <mu1>0.3</mu1>
+            <mu2>0.3</mu2>
+            <kp>10000000.0</kp>
+            <kd>10000.0</kd>
+        </gazebo>
+        <link name="piston_base">
+            <visual name="piston_base_visual">
+                <origin xyz="0 0 0" rpy="0 0 0"/>
+                <geometry>
+                    <cylinder length="${piston_base_width}" radius="${piston_base_radius}"/>
+                </geometry>
+                <material name="grey">
+                    <color rgba="0.2 0.2 0.2 1.0"/>
+                </material>
+            </visual>
+            <collision name="piston_base_collision">
+                <origin xyz="0 0 0" rpy="0 0 0"/>
+                <geometry>
+                    <cylinder length="${piston_base_width}" radius="${piston_base_radius}"/>
+                </geometry>
+            </collision>
+            <inertial>
+                <mass value="${piston_base_mass}" />
+                <origin rpy="0 0 0" xyz="0 0 0" />
+                <inertia ixx="${(2/5) * piston_base_mass * (piston_base_radius * piston_base_radius)}" ixy="0.0" ixz="0.0"
+                        iyy="${(2/5) * piston_base_mass * (piston_base_radius * piston_base_radius)}" iyz="0.0"
+                        izz="${(2/5) * piston_base_mass * (piston_base_radius * piston_base_radius)}" />
+            </inertial>
+        </link>
+        <joint name="joint_base_cylinder" type="fixed">
+                <parent link="piston_cylinder" />
+                <child link="piston_base" />
+                <origin rpy="0 0 0" xyz="0 0 0.08" />
         </joint>
     </xacro:macro>
@@ -152,9 +254,10 @@
     <xacro:traction_wheel_link prefix="left_wheel_link" pos_X="0" pos_Y="0.296395" pos_Z="-0.0118" pos_r="0" pos_p="0" pos_y="1.57" />
     <xacro:traction_wheel_link prefix="right_wheel_link" pos_X="0" pos_Y="-0.296395" pos_Z="-0.0118" pos_r="0" pos_p="0" pos_y="1.57" />
-    <xacro:caster_wheel_link prefix="back_left_caster_wheel_link" pos_X="0.32" pos_Y="0.07" pos_Z="-0.0693" pos_r="-1.57" pos_p="0" pos_y="0" />
-    <xacro:caster_wheel_link prefix="back_right_caster_wheel_link" pos_X="0.32" pos_Y="-0.07" pos_Z="-0.0693" pos_r="-1.57" pos_p="0" pos_y="0" />
-    <xacro:caster_wheel_link prefix="front_left_caster_wheel_link" pos_X="-0.32" pos_Y="0.07" pos_Z="-0.0693" pos_r="-1.57" pos_p="0" pos_y="0" />
-    <xacro:caster_wheel_link prefix="front_right_caster_wheel_link" pos_X="-0.32" pos_Y="-0.07" pos_Z="-0.0693" pos_r="-1.57" pos_p="0" pos_y="0" />
+    <xacro:caster_wheel_link prefix="back_left_caster_wheel_link" pos_X="0.32" pos_Y="0.07" pos_Z="-0.092" pos_r="-1.57" pos_p="0" pos_y="0" />
+    <xacro:caster_wheel_link prefix="back_right_caster_wheel_link" pos_X="0.32" pos_Y="-0.07" pos_Z="-0.092" pos_r="-1.57" pos_p="0" pos_y="0" />
+    <xacro:caster_wheel_link prefix="front_left_caster_wheel_link" pos_X="-0.32" pos_Y="0.07" pos_Z="-0.092" pos_r="-1.57" pos_p="0" pos_y="0" />
+    <xacro:caster_wheel_link prefix="front_right_caster_wheel_link" pos_X="-0.32" pos_Y="-0.07" pos_Z="-0.092" pos_r="-1.57" pos_p="0" pos_y="0" />
     <xacro:tray_link/>
+    <xacro:piston_link/>
     <xacro:imu_sensor/>
     <xacro:laser_sensor

File: ugv_robots_descriptions/robots_description/oni.urdf.xacro (robot description, xacro)
@@ -5,4 +5,7 @@
     <xacro:include filename="controller/omni_drive.urdf.xacro"/>
     <xacro:property name="chassis" value="file:///$(find ugv_robots_descriptions)/robots_description/meshes/oni_meshes/chassis.dae"/>
+    <xacro:property name="left_wheel" value="file:///$(find ugv_robots_descriptions)/robots_description/meshes/oni_meshes/fl_wheel.dae"/>
+    <xacro:property name="right_wheel" value="file:///$(find ugv_robots_descriptions)/robots_description/meshes/oni_meshes/fr_wheel.dae"/>
+    <xacro:property name="base_mass" value="0.8"/>
     <xacro:property name="wheel_radius" value="0.033"/>
     <xacro:property name="wheel_width" value="0.026"/>
@@ -26,5 +29,5 @@
             </collision>
             <inertial>
-                <mass value="0.8"/>
+                <mass value="${base_mass}"/>
                 <origin xyz="0 0 0" rpy="0 0 0" />
                 <inertia ixx="0.0029" ixy="0.0" ixz="0.0" iyy="0.0029" iyz="0.0" izz="0.00533"/>
@@ -68,6 +71,6 @@
         <gazebo reference="${side}_wheel_link">
             <selfCollide>false</selfCollide>
-            <mu1>0.03</mu1>
-            <mu2>0.03</mu2>
+            <mu1>1.5</mu1>
+            <mu2>1.5</mu2>
             <kp>1000000.0</kp>
             <kd>100.0</kd>
@@ -86,5 +89,5 @@
         y_reflect="-1"
         orientation_z="${pi/2}"
-        mesh="file:///$(find ugv_robots_descriptions)/robots_description/meshes/oni_meshes/fr_wheel.dae"
+        mesh="${right_wheel}"
     />
     <xacro:mecanum_wheel_link
@@ -93,5 +96,5 @@
         y_reflect="1"
         orientation_z="${-pi/2}"
-        mesh="file:///$(find ugv_robots_descriptions)/robots_description/meshes/oni_meshes/fl_wheel.dae"
+        mesh="${left_wheel}"
     />
     <xacro:mecanum_wheel_link
@@ -100,5 +103,5 @@
         y_reflect="-1"
         orientation_z="${pi/2}"
-        mesh="file:///$(find ugv_robots_descriptions)/robots_description/meshes/oni_meshes/fr_wheel.dae"
+        mesh="${right_wheel}"
     />
     <xacro:mecanum_wheel_link
@@ -107,5 +110,5 @@
         y_reflect="1"
         orientation_z="${-pi/2}"
-        mesh="file:///$(find ugv_robots_descriptions)/robots_description/meshes/oni_meshes/fl_wheel.dae"
+        mesh="${left_wheel}"
     />
     <xacro:imu_sensor/>
