Commit message: Só falta ajeitar o ekf do l1br

File: ugv_robots_descriptions/robots_description/controller/omni_drive.urdf.xacro (robot description, xacro)
@@ -4,8 +4,9 @@
             <plugin name="omni_drive_controller" filename="libgazebo_ros_planar_move.so">
                 <ros>
-                    <argument>odom:=odom/unfiltered</argument>
+                    <argument>odom:=oni/odom/unfiltered</argument>
+                    <remapping>cmd_vel:=oni/cmd_vel</remapping>
                 </ros>
-                <command_topic>cmd_vel</command_topic>
-                <odometry_topic>odom/unfiltered/</odometry_topic>
+                <command_topic>oni/cmd_vel</command_topic>
+                <odometry_topic>oni/odom/unfiltered</odometry_topic>
                 <odometry_frame>odom</odometry_frame>
                 <odometry_rate>20.0</odometry_rate>

File: ugv_robots_descriptions/robots_description/l1br.urdf.xacro (robot description, xacro)
@@ -41,5 +41,5 @@
             <origin xyz="0  0  0" rpy="0 0 0"/>
             <geometry>
-            <mesh filename="file:///$(find ugv_robots_description)/meshes/l1br_meshes/chassis.dae" />
+            <mesh filename="file:///$(find ugv_robots_descriptions)/robots_description/meshes/l1br_meshes/chassis.dae" />
             </geometry>
         </visual>
@@ -90,5 +90,5 @@
                 <origin rpy="0 0 0" xyz="0 0 0" />
                 <geometry>
-                    <mesh filename="file:///$(find ugv_robots_description)/meshes/wheel.dae" scale="1 1 1" />
+                    <mesh filename="file:///$(find ugv_robots_descriptions)/robots_description/meshes/l1br_meshes/wheel.dae" scale="1 1 1" />
                 </geometry>
             </visual>
@@ -136,5 +136,5 @@
             <origin xyz="0 0 0.0118" rpy="0 0 0"/>
             <geometry>
-                <mesh filename="file:///$(find l1br)/meshes/ELV_conjuntocompleto.dae" scale="1 1 1"/>
+                <mesh filename="file:///$(find ugv_robots_descriptions)/robots_description/meshes/l1br_meshes/tray.dae" scale="1 1 1"/>
             </geometry>
         </visual>
@@ -260,5 +260,7 @@
     <xacro:tray_link/>
     <xacro:piston_link/>
-    <xacro:imu_sensor/>
+    <xacro:imu_sensor
+        topic="l1br/imu/data"
+    />
     <xacro:laser_sensor
         update_rate="5"
@@ -271,4 +273,5 @@
         pos_y="0"
         pos_z="0.188"
+        topic="l1br/scan"
     />
     <xacro:diff_drive_controller

File: ugv_robots_descriptions/robots_description/oni.urdf.xacro (robot description, xacro)
@@ -1,4 +1,4 @@
 <?xml version="1.0"?>
-<robot xmlns:xacro="http://ros.org/wiki/xacro" name="Oni">
+<robot xmlns:xacro="http://ros.org/wiki/xacro" name="oni">
     <xacro:include filename="sensors/imu_sensor.urdf.xacro"/>
     <xacro:include filename="sensors/laser_sensor.urdf.xacro"/>
@@ -35,6 +35,6 @@
         </link>
         <gazebo reference="base_link">
-            <mu1>0.3</mu1>
-            <mu2>0.3</mu2>
+            <mu1>0.01</mu1>
+            <mu2>0.01</mu2>
             <kp>1000000.0</kp>
             <kd>100</kd>
@@ -112,5 +112,7 @@
         mesh="${left_wheel}"
     />
-    <xacro:imu_sensor/>
+    <xacro:imu_sensor
+        topic="oni/imu/data"
+    />
     <xacro:laser_sensor
         update_rate="5"
@@ -123,4 +125,5 @@
         pos_y="0"
         pos_z="0.075"
+        topic="oni/scan"
     />
     <xacro:omni_drive_controller/>

File: ugv_robots_descriptions/robots_description/sensors/imu_sensor.urdf.xacro (robot description, xacro)
@@ -1,4 +1,4 @@
 <robot xmlns:xacro="http://ros.org/wiki/xacro">
-    <xacro:macro name="imu_sensor">
+    <xacro:macro name="imu_sensor" params="topic">
         <link name="imu_link"/>
         <joint name="imu_to_body" type="fixed">
@@ -69,10 +69,9 @@
                 <plugin filename="libgazebo_ros_imu_sensor.so" name="imu_plugin">
                     <ros>
-                        <remapping>~/out:=imu/data</remapping>
-                        <namespace>/oni</namespace>
+                        <remapping>~/out:=${topic}</remapping>
                     </ros>
                     <bodyName>imu_link</bodyName>
                     <frameName>imu_link</frameName>
-                    <topicName>imu/data</topicName>
+                    <topicName>${topic}</topicName>
                     <updateRateHZ>10.0</updateRateHZ>
                     <gaussianNoise>0.0</gaussianNoise>

File: ugv_robots_descriptions/robots_description/sensors/laser_sensor.urdf.xacro (robot description, xacro)
@@ -1,5 +1,5 @@
 <robot xmlns:xacro="http://ros.org/wiki/xacro">
     <xacro:property name="M_PI" value="3.1415926535897931" />
-    <xacro:macro name="laser_sensor" params="update_rate ray_count min_angle max_angle min_range max_range pos_x pos_y pos_z">
+    <xacro:macro name="laser_sensor" params="update_rate ray_count min_angle max_angle min_range max_range pos_x pos_y pos_z topic">
         <link name="laser_link">
             <visual>
@@ -69,8 +69,8 @@
                 <plugin name="base_link_gazebo_ros_head_hokuyo_controller" filename="libgazebo_ros_ray_sensor.so">
                     <ros>
-                        <remapping>~/out:=scan</remapping>
+                        <remapping>~/out:=${topic}</remapping>
                     </ros>
                     <output_type>sensor_msgs/LaserScan</output_type>
-                    <topicName>scan</topicName>
+                    <topicName>${topic}</topicName>
                     <frame_name>laser_link</frame_name>
                     <output_type>sensor_msgs/LaserScan</output_type>
