Commit message: Consertado topico de leitura da descrição do l1br e mudado local de spawn dos robôs em relação ao mapa

File: ugv_robots_descriptions/robots_description/l1br/urdf/sensors/laser_sensor.urdf.xacro (robot description, xacro)
@@ -7,5 +7,5 @@
                 <origin xyz="0 0 -0.025" rpy="0 0 ${M_PI/2}"/>
                 <geometry>
-                    <mesh filename="file:///$(find ugv_robots_descriptions)/robots_description/l1brs/meshes/rplidar.dae"/>
+                    <mesh filename="file:///$(find ugv_robots_descriptions)/robots_description/l1br/meshes/rplidar.dae"/>
                 </geometry>
                 <material name="white">
