Commit message: bandeja e readme

File: ugv_robots_descriptions/robots_description/l1br/urdf/robot_parts/caster_wheel.urdf.xacro (robot description, xacro)
@@ -14,6 +14,6 @@
         <gazebo reference="${prefix}">
             <selfCollide>false</selfCollide>
-            <mu1>0.2</mu1>
-            <mu2>0.2</mu2>
+            <mu1>0.3</mu1>
+            <mu2>0.3</mu2>
             <kp>10000000.0</kp>
             <kd>10000.0</kd>

File: ugv_robots_descriptions/robots_description/l1br/urdf/robot_parts/piston.urdf.xacro (robot description, xacro)
@@ -9,5 +9,5 @@
     <xacro:macro name="piston">
         <gazebo reference="piston_cylinder">
-            <selfCollide>true</selfCollide>
+            <selfCollide>false</selfCollide>
             <mu1>0.1</mu1>
             <mu2>0.1</mu2>
@@ -47,5 +47,5 @@
         </joint>
         <gazebo reference="piston_base">
-            <selfCollide>true</selfCollide>
+            <selfCollide>false</selfCollide>
             <mu1>1</mu1>
             <mu2>1</mu2>

File: ugv_robots_descriptions/robots_description/l1br/urdf/robot_parts/traction_wheel.urdf.xacro (robot description, xacro)
@@ -14,6 +14,6 @@
         <gazebo reference="${prefix}">
             <selfCollide>false</selfCollide>
-            <mu1>1.5</mu1>
-            <mu2>1.5</mu2>
+            <mu1>2</mu1>
+            <mu2>2</mu2>
             <kp>1000000.0</kp>
             <kd>100.0</kd>

File: ugv_robots_descriptions/robots_description/l1br/urdf/robot_parts/tray.urdf.xacro (robot description, xacro)
@@ -29,6 +29,6 @@
         <gazebo reference="tray">
             <selfCollide>true</selfCollide>
-            <mu1 value="1.5" />
-            <mu2 value="1.5" />
+            <mu1 value="2" />
+            <mu2 value="2" />
             <kp value="10000000.0" />
             <kd value="10000" />
@@ -42,9 +42,10 @@
                 <!-- <limit effort="1000.0" lower="0" upper="0.3" velocity="0.5"/> -->
         <!-- </joint> -->
-        <joint name="joint_tray" type="continuous">
+        <joint name="joint_tray" type="revolute">
                 <parent link="piston_base" />
                 <child link="tray" />
                 <origin rpy="0 0 0" xyz="0 0 -0.08" />
                 <axis xyz="0 0 1"/>
+                <limit effort="100" lower="-6" upper="6" velocity="0.1"/>
         </joint>
     </xacro:macro>
