Commit message: consertado bugs no launcher do l1br e modularizado oni

File: ugv_robots_descriptions/robots_description/l1br/urdf/l1br.urdf.xacro (robot description, xacro)
@@ -2,16 +2,18 @@
 <robot name="l1br" xmlns:xacro="http://ros.org/wiki/xacro">
   <!--=========================== CONTROL ===========================-->
-  <xacro:include filename="l1br_control.xacro" />
+  <xacro:include filename="l1br_diff_drive_control.urdf.xacro" />
   <xacro:include filename="sensors/imu_sensor.urdf.xacro" />
   <xacro:include filename="sensors/laser_sensor.urdf.xacro" />
   <!-- =========================== ROBOT ===========================  -->
-  <xacro:include filename="robot_parts/traction_wheel.xacro" />
-  <xacro:include filename="robot_parts/caster_wheel.xacro" />
-  <xacro:include filename="robot_parts/robot_base.xacro" />
-  <xacro:include filename="robot_parts/tray.xacro" />
+  <xacro:include filename="robot_parts/traction_wheel.urdf.xacro" />
+  <xacro:include filename="robot_parts/caster_wheel.urdf.xacro" />
+  <xacro:include filename="robot_parts/robot_base.urdf.xacro" />
+  <xacro:include filename="robot_parts/tray.urdf.xacro" />
+  <xacro:include filename="robot_parts/piston.urdf.xacro" />
   <xacro:tray/>
-  <xacro:include filename="robot_parts/piston.xacro" />
   <xacro:piston/>
-  <xacro:imu_sensor/>
+  <xacro:imu_sensor
+    topic="l1br/imu/data"
+  />
   <xacro:laser_sensor
     update_rate="5"
@@ -21,8 +23,8 @@
     min_range="0.12"
     max_range="8.0"
-    topic_name="scan"
     pos_x="0.27"
     pos_y="0"
     pos_z="0.188"
+    topic="l1br/scan"
   />
 </robot>

File: ugv_robots_descriptions/robots_description/l1br/urdf/robot_parts/robot_base.urdf.xacro (robot description, xacro)
@@ -25,5 +25,5 @@
             <origin xyz="0  0  0" rpy="0 0 0"/>
             <geometry>
-            <mesh filename="file:///$(find l1br)/meshes/EST_estrutura_m3.dae" />
+            <mesh filename="file:///$(find ugv_robots_descriptions)/robots_description/l1br/meshes/chassis.dae" />
             </geometry>
         </visual>

File: ugv_robots_descriptions/robots_description/l1br/urdf/robot_parts/traction_wheel.urdf.xacro (robot description, xacro)
@@ -36,5 +36,5 @@
                 <origin rpy="0 0 0" xyz="0 0 0" />
                 <geometry>
-                    <mesh filename="file:///$(find l1br)/meshes/M_rodatrativa.dae" scale="1 1 1" />
+                    <mesh filename="file:///$(find ugv_robots_descriptions)/robots_description/l1br/meshes/wheel.dae" scale="1 1 1" />
                 </geometry>
             </visual>

File: ugv_robots_descriptions/robots_description/l1br/urdf/robot_parts/tray.urdf.xacro (robot description, xacro)
@@ -10,5 +10,5 @@
             <origin xyz="0 0 0.0118" rpy="0 0 0"/>
             <geometry>
-                <mesh filename="file:///$(find l1br)/meshes/ELV_conjuntocompleto.dae" scale="1 1 1"/>
+                <mesh filename="file:///$(find ugv_robots_descriptions)/robots_description/l1br/meshes/tray.dae" scale="1 1 1"/>
             </geometry>
         </visual>

File: ugv_robots_descriptions/robots_description/l1br/urdf/sensors/imu_sensor.urdf.xacro (robot description, xacro)
@@ -1,5 +1,4 @@
-<?xml version="1.0" ?>
 <robot xmlns:xacro="http://ros.org/wiki/xacro">
-    <xacro:macro name="imu_sensor">
+    <xacro:macro name="imu_sensor" params="topic">
         <link name="imu_link"/>
         <joint name="imu_to_body" type="fixed">
@@ -70,9 +69,9 @@
                 <plugin filename="libgazebo_ros_imu_sensor.so" name="imu_plugin">
                     <ros>
-                        <remapping>~/out:=imu/data</remapping>
+                        <remapping>~/out:=${topic}</remapping>
                     </ros>
                     <bodyName>imu_link</bodyName>
                     <frameName>imu_link</frameName>
-                    <topicName>imu/data</topicName>
+                    <topicName>${topic}</topicName>
                     <updateRateHZ>10.0</updateRateHZ>
                     <gaussianNoise>0.0</gaussianNoise>

File: ugv_robots_descriptions/robots_description/l1br/urdf/sensors/laser_sensor.urdf.xacro (robot description, xacro)
@@ -1,11 +1,10 @@
-<?xml version="1.0" ?>
 <robot xmlns:xacro="http://ros.org/wiki/xacro">
-    <xacro:property name="M_PI" value="3.14159265358979323846264338327950288419716939937510" />
-    <xacro:macro name="laser_sensor" params="update_rate ray_count min_angle max_angle min_range max_range topic_name pos_x pos_y pos_z">
-        <link name="lidar_link">
+    <xacro:property name="M_PI" value="3.1415926535897931" />
+    <xacro:macro name="laser_sensor" params="update_rate ray_count min_angle max_angle min_range max_range pos_x pos_y pos_z topic">
+        <link name="laser_link">
             <visual>
                 <origin xyz="0 0 -0.025" rpy="0 0 ${M_PI/2}"/>
                 <geometry>
-                    <mesh filename="file:///$(find l1br)/meshes/rplidar.dae"/>
+                    <mesh filename="file:///$(find ugv_robots_descriptions)/robots_description/l1brs/meshes/rplidar.dae"/>
                 </geometry>
                 <material name="white">
@@ -27,10 +26,10 @@
             </inertial>
         </link>
-        <joint name="lidar_link_to_base_link" type="fixed">
+        <joint name="base_link_to_base_link" type="fixed">
             <parent link="base_link"/>
-            <child link="lidar_link"/>
+            <child link="laser_link"/>
             <origin xyz="${pos_x} ${pos_y} ${pos_z}" rpy="0 0 0"/>
         </joint>
-        <gazebo reference="lidar_link">
+        <gazebo reference="laser_link">
             <visual>
                 <material>
@@ -42,6 +41,6 @@
             </visual>
         </gazebo>
-        <gazebo reference="lidar_link">
-            <sensor type="ray" name="lidar_link_head_hokuyo_sensor">
+        <gazebo reference="laser_link">
+            <sensor type="ray" name="base_link_head_hokuyo_sensor">
                 <always_on>true</always_on>
                 <update_rate>${update_rate}</update_rate>
@@ -51,8 +50,8 @@
                     <scan>
                         <horizontal>
-                            <samples>${ray_count}</samples>
-                            <resolution>1</resolution>
-                            <min_angle>${min_angle}</min_angle>
-                            <max_angle>${max_angle}</max_angle>
+                        <samples>${ray_count}</samples>
+                        <resolution>1</resolution>
+                        <min_angle>${min_angle}</min_angle>
+                        <max_angle>${max_angle}</max_angle>
                         </horizontal>
                     </scan>
@@ -68,11 +67,12 @@
                     </noise>
                 </ray>
-                <plugin name="lidar_link_gazebo_ros_head_hokuyo_controller" filename="libgazebo_ros_ray_sensor.so">
+                <plugin name="base_link_gazebo_ros_head_hokuyo_controller" filename="libgazebo_ros_ray_sensor.so">
                     <ros>
-                        <remapping>~/out:=${topic_name}</remapping>
+                        <remapping>~/out:=${topic}</remapping>
                     </ros>
                     <output_type>sensor_msgs/LaserScan</output_type>
-                    <topicName>${topic_name}</topicName>
-                    <frame_name>lidar_link</frame_name>
+                    <topicName>${topic}</topicName>
+                    <frame_name>laser_link</frame_name>
+                    <output_type>sensor_msgs/LaserScan</output_type>
                 </plugin>
             </sensor>

File: ugv_robots_descriptions/robots_description/oni/urdf/oni_omni_drive_control.urdf.xacro (robot description, xacro)
@@ -17,3 +17,4 @@
         </gazebo>
     </xacro:macro>
+    <xacro:omni_drive_controller/>
 </robot>

File: ugv_robots_descriptions/robots_description/oni/urdf/robot_parts/traction_wheel.urdf.xacro (robot description, xacro)
@@ -1,11 +1,6 @@
 <?xml version="1.0"?>
 <robot xmlns:xacro="http://ros.org/wiki/xacro" name="oni">
-    <xacro:include filename="sensors/imu_sensor.urdf.xacro"/>
-    <xacro:include filename="sensors/laser_sensor.urdf.xacro"/>
-    <xacro:include filename="controller/omni_drive.urdf.xacro"/>
-    <xacro:property name="chassis" value="file:///$(find ugv_robots_descriptions)/robots_description/meshes/oni_meshes/chassis.dae"/>
-    <xacro:property name="left_wheel" value="file:///$(find ugv_robots_descriptions)/robots_description/meshes/oni_meshes/fl_wheel.dae"/>
-    <xacro:property name="right_wheel" value="file:///$(find ugv_robots_descriptions)/robots_description/meshes/oni_meshes/fr_wheel.dae"/>
-    <xacro:property name="base_mass" value="0.8"/>
+    <xacro:property name="left_wheel" value="file:///$(find ugv_robots_descriptions)/robots_description/oni/meshes/fl_wheel.dae"/>
+    <xacro:property name="right_wheel" value="file:///$(find ugv_robots_descriptions)/robots_description/oni/meshes/fr_wheel.dae"/>
     <xacro:property name="wheel_radius" value="0.033"/>
     <xacro:property name="wheel_width" value="0.026"/>
@@ -14,37 +9,4 @@
     <xacro:property name="wheel_zoff" value="-0.014"/>
     <xacro:property name="wheel_mass" value="0.4"/>
-    <xacro:macro name="base_link">
-        <link name="base_link">
-            <visual>
-                <origin xyz="0 0 0" rpy="0 0 -${pi/2}"/>
-                <geometry>
-                    <mesh filename="${chassis}"/>
-                </geometry>
-            </visual>
-            <collision>
-                <origin xyz="0 0 0" rpy="0 0 -${pi/2}"/>
-                <geometry>
-                    <mesh filename="${chassis}"/>
-                </geometry>
-            </collision>
-            <inertial>
-                <mass value="${base_mass}"/>
-                <origin xyz="0 0 0" rpy="0 0 0" />
-                <inertia ixx="0.0029" ixy="0.0" ixz="0.0" iyy="0.0029" iyz="0.0" izz="0.00533"/>
-            </inertial>
-        </link>
-        <gazebo reference="base_link">
-            <mu1>0.01</mu1>
-            <mu2>0.01</mu2>
-            <kp>1000000.0</kp>
-            <kd>100</kd>
-        </gazebo>
-        <link name="base_footprint"/>
-        <joint name="base_footprint_to_base_link" type="fixed">
-            <parent link="base_link"/>
-            <child link="base_footprint"/>
-            <origin xyz="0.0 0.0 ${-wheel_radius - wheel_zoff}" rpy="0 0 0"/>
-        </joint>
-    </xacro:macro>
     <xacro:macro name="mecanum_wheel_link" params="side x_reflect y_reflect orientation_z mesh">
         <link name="${side}_wheel_link">
@@ -71,6 +33,6 @@
         <gazebo reference="${side}_wheel_link">
             <selfCollide>false</selfCollide>
-            <mu1>1.5</mu1>
-            <mu2>1.5</mu2>
+            <mu1>0.03</mu1>
+            <mu2>0.03</mu2>
             <kp>1000000.0</kp>
             <kd>100.0</kd>
@@ -83,5 +45,4 @@
         </joint>
     </xacro:macro>
-    <xacro:base_link/>
     <xacro:mecanum_wheel_link
         side="front_right"
@@ -112,19 +73,3 @@
         mesh="${left_wheel}"
     />
-    <xacro:imu_sensor
-        topic="oni/imu/data"
-    />
-    <xacro:laser_sensor
-        update_rate="5"
-        ray_count="360"
-        min_angle="0"
-        max_angle="6.28"
-        min_range="0.12"
-        max_range="8.0"
-        pos_x="-0.0475"
-        pos_y="0"
-        pos_z="0.075"
-        topic="oni/scan"
-    />
-    <xacro:omni_drive_controller/>
 </robot>

File: ugv_robots_descriptions/robots_description/oni/urdf/sensors/laser_sensor.urdf.xacro (robot description, xacro)
@@ -6,5 +6,5 @@
                 <origin xyz="0 0 -0.025" rpy="0 0 ${M_PI/2}"/>
                 <geometry>
-                    <mesh filename="file:///$(find ugv_robots_descriptions)/robots_description/meshes/rplidar.dae"/>
+                    <mesh filename="file:///$(find ugv_robots_descriptions)/robots_description/oni/meshes/rplidar.dae"/>
                 </geometry>
                 <material name="white">

Commit message: fix scan and other features

File: ugv_robots_descriptions/robots_description/l1br/urdf/l1br.urdf.xacro (robot description, xacro)
@@ -26,5 +26,5 @@
     pos_y="0"
     pos_z="0.188"
-    topic="l1br/scan"
+    topic="/l1br/scan"
   />
 </robot>

File: ugv_robots_descriptions/robots_description/l1br/urdf/l1br_diff_drive_control.urdf.xacro (robot description, xacro)
@@ -19,7 +19,9 @@
       <robotBaseFrame>base_link</robotBaseFrame>
       <odometrySource>1</odometrySource>
-      <publishWheelTF>true</publishWheelTF>
+      <publishWheelTF>false</publishWheelTF>
       <publishOdom>true</publishOdom>
-      <publishWheelJointState>true</publishWheelJointState>
+      <publishOdomTF>true</publishOdomTF>
+      <publishWheelJointState>false</publishWheelJointState>
+      <publishTF>1</publishTF>
       <legacyMode>true</legacyMode>
     </plugin>

File: ugv_robots_descriptions/robots_description/l1br/urdf/sensors/laser_sensor.urdf.xacro (robot description, xacro)
@@ -13,5 +13,5 @@
                 </material>
             </visual>
-            <collision>
+            <!-- <collision>
                 <origin xyz="0.003 -0.003 -0.027" rpy="0 0 ${M_PI/2}"/>
                 <geometry>
@@ -25,12 +25,12 @@
                         iyy="${(2/5) * 0.1 * (0.0375 * 0.0375)}" iyz="0"
                         izz="${(2/5) * 0.1 * (0.0375 * 0.0375)}" />
-            </inertial>
+            </inertial> -->
         </link>
-        <joint name="base_link_to_base_link" type="fixed">
+        <joint name="laser_link_to_base_link" type="fixed">
             <parent link="base_link"/>
             <child link="laser_link"/>
             <origin xyz="${pos_x} ${pos_y} ${pos_z}" rpy="0 0 0"/>
         </joint>
-        <gazebo reference="laser_link">
+        <!-- <gazebo reference="laser_link">
             <visual>
                 <material>
@@ -41,11 +41,11 @@
                 </material>
             </visual>
-        </gazebo>
+        </gazebo> -->
         <gazebo reference="laser_link">
-            <sensor type="ray" name="base_link_head_hokuyo_sensor">
+            <sensor type="ray" name="laser_link_head_hokuyo_sensor">
                 <always_on>true</always_on>
                 <update_rate>${update_rate}</update_rate>
-                <pose>0 0 0 0 0 0</pose>
-                <visualize>false</visualize>
+                <!-- <pose>0 0 0 0 0 0</pose> -->
+                <visualize>true</visualize>
                 <ray>
                     <scan>
@@ -68,11 +68,11 @@
                     </noise>
                 </ray>
-                <plugin name="base_link_gazebo_ros_head_hokuyo_controller" filename="libgazebo_ros_ray_sensor.so">
-                    <ros>
+                <plugin name="laser_link_gazebo_ros_head_hokuyo_controller" filename="libgazebo_ros_laser.so">
+                    <!-- <ros>
                         <remapping>~/out:=${topic}</remapping>
-                    </ros>
+                    </ros> -->
                     <output_type>sensor_msgs/LaserScan</output_type>
                     <topicName>${topic}</topicName>
-                    <frame_name>laser_link</frame_name>
+                    <frameName>laser_link</frameName>
                     <output_type>sensor_msgs/LaserScan</output_type>
                 </plugin>
