Commit message: fixed laser_scan to oni

File: ugv_robots_descriptions/robots_description/oni/urdf/oni_omni_drive_control.urdf.xacro (robot description, xacro)
@@ -1,3 +1,3 @@
-<?xml version="1.0 ?>
+<?xml version="1.0" ?>
 <robot name="oni" xmlns:xacro="http://ros.org/wiki/xacro">
     <xacro:macro name="omni_drive_controller">

File: ugv_robots_descriptions/robots_description/oni/urdf/sensors/laser_sensor.urdf.xacro (robot description, xacro)
@@ -1,2 +1,3 @@
+<?xml version="1.0" ?>
 <robot xmlns:xacro="http://ros.org/wiki/xacro">
     <xacro:property name="M_PI" value="3.1415926535897931" />
@@ -12,5 +13,5 @@
                 </material>
             </visual>
-            <collision>
+            <!-- <collision>
                 <origin xyz="0.003 -0.003 -0.027" rpy="0 0 ${M_PI/2}"/>
                 <geometry>
@@ -24,12 +25,12 @@
                         iyy="${(2/5) * 0.1 * (0.0375 * 0.0375)}" iyz="0"
                         izz="${(2/5) * 0.1 * (0.0375 * 0.0375)}" />
-            </inertial>
+            </inertial> -->
         </link>
-        <joint name="base_link_to_base_link" type="fixed">
+        <joint name="laser_link_to_base_link" type="fixed">
             <parent link="base_link"/>
             <child link="laser_link"/>
             <origin xyz="${pos_x} ${pos_y} ${pos_z}" rpy="0 0 0"/>
         </joint>
-        <gazebo reference="laser_link">
+        <!-- <gazebo reference="laser_link">
             <visual>
                 <material>
@@ -40,11 +41,11 @@
                 </material>
             </visual>
-        </gazebo>
+        </gazebo> -->
         <gazebo reference="laser_link">
-            <sensor type="ray" name="base_link_head_hokuyo_sensor">
+            <sensor type="ray" name="laser_link_head_hokuyo_sensor">
                 <always_on>true</always_on>
                 <update_rate>${update_rate}</update_rate>
-                <pose>0 0 0 0 0 0</pose>
-                <visualize>false</visualize>
+                <!-- <pose>0 0 0 0 0 0</pose> -->
+                <visualize>true</visualize>
                 <ray>
                     <scan>
@@ -67,5 +68,5 @@
                     </noise>
                 </ray>
-                <plugin name="base_link_gazebo_ros_head_hokuyo_controller" filename="libgazebo_ros_ray_sensor.so">
+                <plugin name="laser_link_gazebo_ros_head_hokuyo_controller" filename="libgazebo_ros_laser.so">
                     <ros>
                         <remapping>~/out:=${topic}</remapping>
@@ -73,5 +74,5 @@
                     <output_type>sensor_msgs/LaserScan</output_type>
                     <topicName>${topic}</topicName>
-                    <frame_name>laser_link</frame_name>
+                    <frameName>laser_link</frameName>
                     <output_type>sensor_msgs/LaserScan</output_type>
                 </plugin>
